Commit message: changed kp to 500 and kd to 20, also added extra reward terms

File: rl-training-genesis/models/g1_12dof.urdf (robot description, URDF)
Before this commit: robot g1_12dof, 31 links, 30 joints
Joints:
- joint left_elbow_joint: type revolute -> fixed
- joint left_shoulder_pitch_joint: type revolute -> fixed
- joint left_shoulder_roll_joint: type revolute -> fixed
- joint left_shoulder_yaw_joint: type revolute -> fixed
- joint left_wrist_roll_joint: type revolute -> fixed
