Commit message: Add VLA manipulation setup and comprehensive documentation
- Updated README with complete project overview and quick start guide
- Added comprehensive documentation in docs/ directory
- Added feb8_demo/ scripts for G1 testing and demonstrations
- Added g1_manipulation/ environment for manipulation tasks
- Modified g1_12dof.urdf to fix left arm joints
- Added g1_23dof.urdf robot model variant
- Updated .gitignore to exclude vla_env/ and outputs/

Co-authored-by: Cursor <cursoragent@cursor.com>

File: rl-training-genesis/models/g1_23dof.urdf (robot description, URDF)
Before this commit: robot g1_12dof, 31 links, 30 joints
Links:
- added link waist_support_link, mass 0.001; collision mesh filename=meshes/waist_support_link.STL; visual mesh filename=meshes/waist_support_link.STL
- added link waist_yaw_fixed_link, mass 0.244; visual mesh filename=meshes/waist_yaw_link.STL
- link torso_link: mass 6.78 -> 8.562; geometry collision mesh filename=meshes/torso_link.STL; visual mesh filename=meshes/torso_link.STL
Joints:
- added joint waist_support_joint: type fixed, parent torso_link, child waist_support_link, origin xyz=0.0039635 0 -0.054 rpy=0 0 0
- added joint waist_yaw_fixed_joint: type fixed, parent torso_link, child waist_yaw_fixed_link, origin xyz=0.0039635 0 -0.054 rpy=0 0 0
- joint d435_joint: origin xyz=0.0576235 0.01753 0.42987 rpy=0 0.8307767239493009 0 -> xyz=0.0576235 0.01753 0.41987 rpy=0 0.8307767239493009 0
- joint head_joint: origin xyz=0.0039635 0 -0.044 rpy=0 0 0 -> xyz=0.0039635 0 -0.054 rpy=0 0 0
- joint imu_in_torso_joint: origin xyz=-0.03959 -0.00224 0.14792 rpy=0 0 0 -> xyz=-0.03959 -0.00224 0.13792 rpy=0 0 0
- joint left_elbow_joint: type fixed -> revolute
- joint left_hip_roll_joint: limit lower=-0.5236 upper=2.9671 effort=139 velocity=20 -> lower=-0.5236 upper=2.9671 effort=88 velocity=32
- joint left_shoulder_pitch_joint: origin xyz=0.0039563 0.10022 0.24778 rpy=0.27931 5.4949E-05 -0.00019159 -> xyz=0.0039563 0.10022 0.23778 rpy=0.27931 5.4949E-05 -0.00019159; type fixed -> revolute
- joint left_shoulder_roll_joint: type fixed -> revolute
- joint left_shoulder_yaw_joint: type fixed -> revolute
- joint left_wrist_roll_joint: type fixed -> revolute
- joint logo_joint: origin xyz=0.0039635 0 -0.044 rpy=0 0 0 -> xyz=0.0039635 0 -0.054 rpy=0 0 0
- joint mid360_joint: origin xyz=0.0002835 0.00003 0.41618 rpy=0 0.04014257279586953 0 -> xyz=0.0002835 0.00003 0.40618 rpy=0 0.04014257279586953 0
- joint right_elbow_joint: type fixed -> revolute
- joint right_hip_roll_joint: limit lower=-2.9671 upper=0.5236 effort=139 velocity=20 -> lower=-2.9671 upper=0.5236 effort=88 velocity=32
- joint right_shoulder_pitch_joint: origin xyz=0.0039563 -0.10021 0.24778 rpy=-0.27931 5.4949E-05 0.00019159 -> xyz=0.0039563 -0.10021 0.23778 rpy=-0.27931 5.4949E-05 0.00019159; type fixed -> revolute
- joint right_shoulder_roll_joint: type fixed -> revolute
- joint right_shoulder_yaw_joint: type fixed -> revolute
- joint right_wrist_roll_joint: type fixed -> revolute
- joint waist_yaw_joint: origin xyz=-0.0039635 0 0.044 rpy=0 0 0 -> xyz=-0.0039635 0 0.054 rpy=0 0 0; type fixed -> revolute
